File: pcb/chocofi-topplate.kicad_pcb (KiCad board)
At the start: 2 copper layers, 111.4 x 90 mm, 23 parts, among them SW10 SW_PUSH, SW11 SW_PUSH, SW12 SW_PUSH, SW14 SW_PUSH, SW15 SW_PUSH, SW16 SW_PUSH, SW17 SW_PUSH, SW18 SW_PUSH, SW19 SW_PUSH, SW2 SW_PUSH, SW20 SW_PUSH, SW21 SW_PUSH, SW3 SW_PUSH, SW4 SW_PUSH, SW5 SW_PUSH, SW6 SW_PUSH, SW8 SW_PUSH, SW9 SW_PUSH

Commit message: Stripes pattern for plate.
Parts:
- added svg2mod: G***, kbd:lines, F.Cu at (108.2, 78.4)
- added svg2mod: G***, kbd:lines-mirrored, B.Cu at (108.1, 78.5)
Other:
- board text removed: "chocofi @pashutk"
